Commit message: testing out dual arm

File: universal_robot/ur_description/urdf/inc/ur_macro.xacro (robot description, xacro)
@@ -316,4 +316,11 @@
       <child link="${prefix}tool0"/>
     </joint>
+   <!-- world environment .xacro if we have one
+    <link name="world" />
+    <joint name="world_to_pick" type="fixed">
+      <parent link="world" />
+      <child link = "${prefix}base_link" />
+      <origin xyz="-0.5 0 0" rpy="0.0 0.0 0.0" />
+    </joint>-->
   </xacro:macro>
 </robot>

File: universal_robot/ur_description/urdf/ur.xacro (robot description, xacro)
@@ -3,9 +3,36 @@
    <!-- import main macro -->
    <xacro:include filename="$(find ur_description)/urdf/inc/ur_macro.xacro"/>
-   <!-- parameters -->
+   <!-- parameters
    <xacro:arg name="joint_limit_params" default=""/>
    <xacro:arg name="kinematics_params" default=""/>
    <xacro:arg name="physical_params" default=""/>
    <xacro:arg name="visual_params" default=""/>
+   -->
+   <!-- legal values:
+         - hardware_interface/PositionJointInterface
+         - hardware_interface/VelocityJointInterface
+         - hardware_interface/EffortJointInterface
+   <xacro:arg name="transmission_hw_interface" default="hardware_interface/PositionJointInterface"/>
+   <xacro:arg name="safety_limits" default="false"/>
+   <xacro:arg name="safety_pos_margin" default="0.15"/>
+   <xacro:arg name="safety_k_position" default="20"/>
+   -->
+   <!-- arm
+   <xacro:ur_robot
+     prefix=""
+     joint_limits_parameters_file="$(arg joint_limit_params)"
+     kinematics_parameters_file="$(arg kinematics_params)"
+     physical_parameters_file="$(arg physical_params)"
+     visual_parameters_file="$(arg visual_params)"
+     transmission_hw_interface="$(arg transmission_hw_interface)"
+     safety_limits="$(arg safety_limits)"
+     safety_pos_margin="$(arg safety_pos_margin)"
+     safety_k_position="$(arg safety_k_position)"/>
+   -->
+   <xacro:arg name="joint_limit_params" default=""/>
+   <xacro:arg name="kinematics_params" default=""/>
+   <xacro:arg name="physical_params" default=""/>
+   <xacro:arg name="visual_params" default=""/>
+   <xacro:arg name="prefix" default=""/>
    <!-- legal values:
          - hardware_interface/PositionJointInterface
@@ -19,5 +46,5 @@
    <!-- arm -->
    <xacro:ur_robot
-     prefix=""
+     prefix="$(arg prefix)"
      joint_limits_parameters_file="$(arg joint_limit_params)"
      kinematics_parameters_file="$(arg kinematics_params)"
