Commit message: dual robot communication setup

File: universal_robot/ur_description/urdf/dispense.xacro (robot description, xacro)
@@ -9,5 +9,5 @@
   <joint name="world_to_dispense" type="fixed">
     <parent link="world" />
-    <child link = "dispense_base_link" />
+    <child link = "$(arg prefix)base_link" />
     <origin xyz="-1.5 0 0" rpy="0.0 0.0 0.0" />
   </joint>

File: universal_robot/ur_description/urdf/dispense_final.xacro (robot description, xacro)
@@ -3,13 +3,35 @@
 <robot xmlns:xacro="http://wiki.ros.org/xacro" name="ur5e_robot">
  <!-- load the urdf file -->
-  <xacro:include filename="$(find ur_description)/urdf/inc/ur5e_macro.xacro"/>
+  <xacro:include filename="$(find ur_description)/urdf/inc/ur_macro.xacro"/>
    <!-- arm 2 -->
-  <xacro:ur5e_robot prefix="" joint_limits_parameters_file="false" kinematics_parameters_file="$(find ur_description)/config/ur5e/kinematic_dispense.yaml"/>
+  <xacro:macro name="ur5e_robot" params="
+   tf_prefix:='hahha'
+   joint_limits_parameters_file:='$(find ur_description)/config/ur5e/joint_limits.yaml'
+   kinematics_parameters_file:='$(find ur_description)/config/ur5e/kinematics_dispense.yaml'
+   physical_parameters_file:='$(find ur_description)/config/ur5e/physical_parameters.yaml'
+   visual_parameters_file:='$(find ur_description)/config/ur5e/visual_parameters.yaml'
+   transmission_hw_interface:=hardware_interface/PositionJointInterface
+   safety_limits:=false
+   safety_pos_margin:=0.15
+   safety_k_position:=20"
+  >
+    <xacro:ur_robot
+      prefix="${prefix}"
+      joint_limits_parameters_file="${joint_limits_parameters_file}"
+      kinematics_parameters_file="${kinematics_parameters_file}"
+      physical_parameters_file="${physical_parameters_file}"
+      visual_parameters_file="${visual_parameters_file}"
+      transmission_hw_interface="${transmission_hw_interface}"
+      safety_limits="${safety_limits}"
+      safety_pos_margin="${safety_pos_margin}"
+      safety_k_position="${safety_k_position}"
+    />
    <!-- world environment .xacro if we have one -->
   <link name="world" />
-  <joint name="world_joint" type="fixed">
+  <joint name="world_to_pick" type="fixed">
     <parent link="world" />
-    <child link = "base_link" />
-    <origin xyz="-1.5 0 0" rpy="0.0 0.0 0.0" />
+    <child link = "$(arg tf_prefix)base_link" />
+    <origin xyz="-3.5 0 0" rpy="0.0 0.0 0.0" />
   </joint>
+  </xacro:macro>
 </robot>

File: universal_robot/ur_description/urdf/pp.xacro (robot description, xacro)
@@ -6,10 +6,11 @@
  -->
   <!-- arm pick and place-->
-  <xacro:ur5e_robot prefix="pickAndPlace_" kinematics_parameters_file="$(find ur_description)/config/ur5e/kinematic_pick_and_place.yaml" />
+  <xacro:ur5e_robot prefix="pickAndPlace_" kinematics_parameters_file="$(find ur_description)/config/ur5e/kinematic_pick_and_place.yaml"
+/>
    <!-- world environment .xacro if we have one -->
   <link name="world" />
   <joint name="world_to_pick" type="fixed">
     <parent link="world" />
-    <child link = "pickAndPlace_base_link" />
+    <child link = "$(arg prefix)base_link" />
     <origin xyz="-0.5 0 0" rpy="0.0 0.0 0.0" />
   </joint>
